File: DesignBlocks/Library.kicad_blocks/RP2354A.kicad_block/RP2354A.kicad_sch (KiCad schematic)
At the start: 28 parts, among them J3 USB_B_Micro, J5 SWD, U4 TLV74311PDBVR, U5 RP2354A-QFN60, Y1 12MHz

Commit message: - Moved the design blocks out from the models directory.
Parts:
- renumbered C25 to C1, C15 to C10, C16 to C11, C17 to C12, C18 to C13, C19 to C14, C26 to C2, C13 to C3, C20 to C4, C12 to C5, C11 to C6, C10 to C7, C55 to C8, C14 to C9, J5 to J1, J3 to J2, R22 to R1, R12 to R2, R6 to R3, R11 to R4, R21 to R5, R8 to R6, R9 to R7, U4 to U1, U5 to U2
Other:
- moved on the sheet: C1, C10, C11, C12, C13, C14, C2, C3, C4, C5, C6, C7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
