File: DesignBlocks/Library.kicad_blocks/iCE40hx1k_vq100.kicad_block/iCE40hx1k_vq100.kicad_pcb (KiCad board)
At the start: 2 copper layers, 27 parts, among them U2 MIC5504-1.2YM5, U3 iCE40HX1K-VQ100

Commit message: - Moved the design blocks out from the models directory.
Parts:
- removed C21, C22, C23, C24, C36, C37, C38, C39, C40: 100nf, Capacitor_SMD:C_0603_1608Metric
- removed D2: D_Dual_Series_ACK, Package_TO_SOT_SMD:SOT-23
- removed R13: 10k, Resistor_SMD:R_0603_1608Metric
- removed R14, R72, R73, R74: 27R, Resistor_SMD:R_0603_1608Metric
- removed U3: iCE40HX1K-VQ100, Package_QFP:LQFP-100_14x14mm_P0.5mm
- added C1: 100nf, Capacitor_SMD:C_0603_1608Metric, B.Cu at (157.1, 121.8)
- added C10: 100nf, Capacitor_SMD:C_0603_1608Metric, B.Cu at (153.7, 113.3)
- added C11: 100nf, Capacitor_SMD:C_0603_1608Metric, B.Cu at (169.2, 114.4)
- added C12: 100nf, Capacitor_SMD:C_0603_1608Metric, B.Cu at (163.1, 109.5)
- added C13: 100nf, Capacitor_SMD:C_0603_1608Metric, B.Cu at (156.6, 109.3)
- added C14: 100nf, Capacitor_SMD:C_0603_1608Metric, B.Cu at (160.0, 106.3)
- added C15: 100nf, Capacitor_SMD:C_0603_1608Metric, B.Cu at (163.1, 106.3)
- added C6: 100nf, Capacitor_SMD:C_0603_1608Metric, B.Cu at (159.6, 118.9)
- added C7: 100nf, Capacitor_SMD:C_0603_1608Metric, B.Cu at (153.7, 116.8)
- added D1: D_Dual_Series_ACK, Package_TO_SOT_SMD:SOT-23, B.Cu at (153.9, 103.5)
- added R1: 10k, Resistor_SMD:R_0603_1608Metric, F.Cu at (177.0, 111.5)
- added R5: 27R, Resistor_SMD:R_0603_1608Metric, F.Cu at (177.0, 108.5)
- added R6: 27R, Resistor_SMD:R_0603_1608Metric, F.Cu at (177.0, 110.0)
- added R7: 10k, Resistor_SMD:R_0603_1608Metric, B.Cu at (168.4, 106.3)
- added R8: 27R, Resistor_SMD:R_0603_1608Metric, F.Cu at (181.3, 115.7)
- added U1: iCE40HX1K-VQ100, Package_QFP:LQFP-100_14x14mm_P0.5mm, F.Cu at (161.3, 114.1)
- C5: value 100nf -> 4.7uf
- C8: value 4.7uf -> 100nf
- R2: value 10k -> 2k2
- R3: value 2k2 -> 27R
- moved CDone1 125.9 mm to (177.1, 115.7), turned to 180 degrees
- moved R4 124.4 mm to (177.0, 107.0), turned to 180 degrees
- moved R3 121.9 mm to (177.0, 105.5), turned to 180 degrees
- moved C8 121.6 mm to (169.2, 117.4), turned to 90 degrees
- moved R2 121.2 mm to (177.0, 112.9), turned to 180 degrees
- moved C2 120.9 mm to (162.3, 121.8), turned to 0 degrees
- moved C3 117.6 mm to (165.3, 121.8), turned to 180 degrees
- moved C4 113.5 mm to (169.2, 108.8), turned to 90 degrees
- moved C5 110.7 mm to (162.4, 115.3), turned to 90 degrees
- moved U2 110.3 mm to (159.2, 113.6), turned to 0 degrees
- moved C9 109.9 mm to (166.2, 114.8), turned to 90 degrees
Connections:
- C2 pad 1: +1V2 -> +3V3
- C3 pad 1: +1V2 -> +3V3
- C4 pad 1: +1V2 -> GND
- C4 pad 2: GND -> +3V3
- C5 pad 1: +1V2 -> GND
- C5 pad 2: GND -> +1V2
- C8 pad 1: GND -> +3V3
- C8 pad 2: +1V2 -> GND
- C9 pad 1: GND -> +1V2
- C9 pad 2: +3V3 -> GND
- R2 pad 2: /~{3v3_RESET} -> /iCE40-CDONE
- R3 pad 1: +3V3 -> unconnected-(R3-Pad1)
- R3 pad 2: /iCE40-CDONE -> /~{iCE40-SS}
- R4 pad 1: Net-(CDone1-K) -> unconnected-(R4-Pad1)
- R4 pad 2: GND -> /iCE40-SCK
Routing:
- net Net-(D1-K): track 0.00 -> 4.40 mm, vias 0 -> 2
- net GND: track 45.8 -> 48.9 mm, vias 35 -> 37
- net Net-(D2-K): track 3.02 -> 0.00 mm, vias 1 -> 0
- net unconnected-(U3D-IOL_10A-Pad20): track 1.05 -> 0.00 mm
- net unconnected-(U3A-IOT_74-Pad79): track 1.05 -> 0.00 mm
- net unconnected-(U1D-IOL_10A-Pad20): track 0.00 -> 1.05 mm
- net unconnected-(U1A-IOT_74-Pad79): track 0.00 -> 1.05 mm
- net unconnected-(U3A-IOT_84_GBIN1-Pad89): track 0.99 -> 0.00 mm
- net unconnected-(U1A-IOT_84_GBIN1-Pad89): track 0.00 -> 0.99 mm
- net unconnected-(U3D-IOL_7B-Pad16): track 0.96 -> 0.00 mm
- net unconnected-(U1D-IOL_7B-Pad16): track 0.00 -> 0.96 mm
- net unconnected-(U1D-IOL_6B_GBIN7-Pad13): track 0.00 -> 0.95 mm
- net unconnected-(U3D-IOL_6B_GBIN7-Pad13): track 0.95 -> 0.00 mm
- net unconnected-(U3C-IOB_36_GBIN4-Pad34): track 0.95 -> 0.00 mm
- net unconnected-(U1C-IOB_36_GBIN4-Pad34): track 0.00 -> 0.95 mm
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