File: DesignBlocks/Library.kicad_blocks/iCE40hx1k_vq100.kicad_block/iCE40hx1k_vq100.kicad_sch (KiCad schematic)
At the start: 27 parts, among them U2 MIC5504-1.2YM5, U3 iCE40HX1K-VQ100

Commit message: - Moved the design blocks out from the models directory.
Parts:
- renumbered C36 to C1, C23 to C10, C39 to C11, C4 to C12, C5 to C13, C21 to C14, C22 to C15, C37 to C2, C38 to C3, C9 to C4, C8 to C5, C2 to C6, C24 to C7, C40 to C8, C3 to C9, D2 to D1, R2 to R1, R3 to R2, R14 to R3, R74 to R4, R72 to R5, R73 to R6, R13 to R7, R4 to R8, U3 to U1
Other:
- moved on the sheet: C1, C10, C11, C12, C13, C14, C15, C2, C3, C4, C5, C6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
